File: pixie2.kicad_sch (KiCad schematic)
At the start: 45 parts, among them J1 Conn_Coaxial, J2 AudioJack2, Q1 BC547, Q2 2N2219, SW1 SW_Push, U1 LM386, Y1 3579kHz

Commit message: fix vcc line
Parts:
- D3: footprint Diode_THT:D_DO-35_SOD27_P5.08mm_Vertical_KathodeUp -> Diode_THT:D_DO-35_SOD27_P2.54mm_Vertical_KathodeUp
- R1, R3: footprint Resistor_THT:R_Axial_DIN0204_L3.6mm_D1.6mm_P5.08mm_Horizontal -> Resistor_THT:R_Axial_DIN0204_L3.6mm_D1.6mm_P2.54mm_Vertical
Changed lines of the file:
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@@
     (property "Reference" "D3" (id 0) (at 102.87 97.9002 0))
     (property "Value" "1N4148" (id 1) (at 102.87 100.4371 0))
-    (property "Footprint" "Diode_THT:D_DO-35_SOD27_P5.08mm_Vertical_KathodeUp" (id 2) (at 102.87 102.87 0)
+    (property "Footprint" "Diode_THT:D_DO-35_SOD27_P2.54mm_Vertical_KathodeUp" (id 2) (at 102.87 102.87 0)
       (effects (font (size 1.27 1.27)) hide)
     )
@@
     (property "Reference" "R1" (id 0) (at 75.565 72.1192 90))
     (property "Value" "10k" (id 1) (at 75.565 74.6561 90))
-    (property "Footprint" "Resistor_THT:R_Axial_DIN0204_L3.6mm_D1.6mm_P5.08mm_Horizontal" (id 2) (at 75.565 78.613 90)
+    (property "Footprint" "Resistor_THT:R_Axial_DIN0204_L3.6mm_D1.6mm_P2.54mm_Vertical" (id 2) (at 75.565 78.613 90)
       (effects (font (size 1.27 1.27)) hide)
     )
@@
       (effects (font (size 1.27 1.27)) (justify left))
     )
-    (property "Footprint" "Resistor_THT:R_Axial_DIN0204_L3.6mm_D1.6mm_P5.08mm_Horizontal" (id 2) (at 98.552 65.405 90)
+    (property "Footprint" "Resistor_THT:R_Axial_DIN0204_L3.6mm_D1.6mm_P2.54mm_Vertical" (id 2) (at 98.552 65.405 90)
       (effects (font (size 1.27 1.27)) hide)
     )
@@
     )
     (path "/52c94579-b45c-445c-ba08-42ddab26390a"
-      (reference "D3") (unit 1) (value "1N4148") (footprint "Diode_THT:D_DO-35_SOD27_P5.08mm_Vertical_KathodeUp")
+      (reference "D3") (unit 1) (value "1N4148") (footprint "Diode_THT:D_DO-35_SOD27_P2.54mm_Vertical_KathodeUp")
     )
     (path "/14661244-47a5-446e-94d8-446808dfc46f"
@@
     )
     (path "/c679ff8e-a3b7-4479-836b-462a3dd7ef0c"
-      (reference "R1") (unit 1) (value "10k") (footprint "Resistor_THT:R_Axial_DIN0204_L3.6mm_D1.6mm_P5.08mm_Horizontal")
+      (reference "R1") (unit 1) (value "10k") (footprint "Resistor_THT:R_Axial_DIN0204_L3.6mm_D1.6mm_P2.54mm_Vertical")
     )
     (path "/f499b87d-4dce-4e6c-9169-f637a600dc96"
@@
     )
     (path "/f53ba1ed-bb18-4dbe-a067-69dda2e4e8ea"
-      (reference "R3") (unit 1) (value "100k") (footprint "Resistor_THT:R_Axial_DIN0204_L3.6mm_D1.6mm_P5.08mm_Horizontal")
+      (reference "R3") (unit 1) (value "100k") (footprint "Resistor_THT:R_Axial_DIN0204_L3.6mm_D1.6mm_P2.54mm_Vertical")
     )
     (path "/4467688f-009a-41f4-ad76-547ce1f27c5b"

Commit message: Finalize
Parts:
- L4: footprint Inductor_THT:L_Axial_L7.0mm_D3.3mm_P10.16mm_Horizontal_Fastron_MICC -> Inductor_THT:L_Axial_L7.0mm_D3.3mm_P5.08mm_Vertical_Fastron_MICC
Changed lines of the file:
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@@
     (property "Reference" "L4" (id 0) (at 179.07 40.2422 90))
     (property "Value" "2u2" (id 1) (at 179.07 42.7791 90))
-    (property "Footprint" "Inductor_THT:L_Axial_L7.0mm_D3.3mm_P10.16mm_Horizontal_Fastron_MICC" (id 2) (at 179.07 44.45 0)
+    (property "Footprint" "Inductor_THT:L_Axial_L7.0mm_D3.3mm_P5.08mm_Vertical_Fastron_MICC" (id 2) (at 179.07 44.45 0)
       (effects (font (size 1.27 1.27)) hide)
     )
@@
     )
     (path "/02bbdd62-5160-4932-b1d2-cf5e5771ab93"
-      (reference "L4") (unit 1) (value "2u2") (footprint "Inductor_THT:L_Axial_L7.0mm_D3.3mm_P10.16mm_Horizontal_Fastron_MICC")
+      (reference "L4") (unit 1) (value "2u2") (footprint "Inductor_THT:L_Axial_L7.0mm_D3.3mm_P5.08mm_Vertical_Fastron_MICC")
     )
     (path "/74689544-f28e-447c-99c3-309831032263"
